File: schematics/sch/tapecleaner.sch (EAGLE design)
At the start: 8 parts, among them U1 GP1A57HR, U2 LOGO-SFESK, U3 GP1A57HR

Commit message: removed .brd file, updated schematic
Parts:
- removed PCB1: ARDUINO_UNO, E14_Arduino_revB:ARDUINO_UNO
- added BRAKE-A_DISABLE, BRAKE-B_DISABLE, SNS0-ENABLE, SNS1_ENABLE, VIN-CONNECT: (no value), jumper:SJ
- added C1, C12, C2, C3, C4, C6, C7, C8: 100n, SmartPrj:C-EUC0603
- added C10, C11, C5, C9: 10u 35V, SmartPrj:C-EUC1210
- added D1, D10, D2, D3, D4, D5, D6, D7, D8, D9: SS14, SmartPrj:SS14
- added FID1, FID2, FID3: FIDUCIALMOUNT, SmartPrj:FIDUCIALMOUNT
- added IC1: L298P, SmartPrj:L298P
- added IC2: 4077D, 40xx:4077D
- added IC4: LMV358MMX, linear:LMV358MMX
- added IN2, IN3: white, SmartPrj:MTA03-100
- added JANALOG: 6x1F-H8.5-L14.5mm, SmartPrj:PINHD-1X6TH
- added JHIGH: 10x1F-H8.5-L14.5mm, SmartPrj:PINHD-1X10TH
- added JLOW, POWER: 8x1F-H8.5-L14.5mm, SmartPrj:PINHD-1X8TH
- added JP3: (no value), SparkFun:M03PTH
- added LED1, LED2, LED3, LED4: Yellow, led:LEDCHIPLED_0805
- added LSP1, LSP2, LSP3, LSP4, LSP5, LSP6: LSP13, solpad:LSP13
- added OUT5, OUT6: orange, SmartPrj:MTA03-100
- added R3, R4, R5: 220, SparkFun:RESISTORPTH1
- added RESET: TS42, SmartPrj:TS42
- added RN1, RN2: 10K, resistor-dil:4R-NCAY16
- added RN3: 1K, resistor-dil:4R-NCAY16
- added TWI-IN, TWI-OUT: (no value), con-amp:MTA04-100
- added U4: GP1A57HR, SparkFun:GP1A57HR
- R1, R2: value 220 -> 0R15; device SparkFun:RESISTORPTH1 -> SmartPrj:R-EU_R1206
Connections:
- new net +3V3: POWER.4
- new net +5V: C1.1, C12.1, C2.1, C3.1, C4.1, C5.1, C6.1, C7.1, C8.1, IC1.VSS, IC2B.I0, IC2B.I1, IC2P.VDD, IC4P.V+, IN2.3, IN3.3, OUT5.3, OUT6.3, POWER.5, TWI-IN.2, TWI-OUT.2
- new net 5: JLOW.6, OUT5.2
- new net 6: JLOW.7, OUT6.2
- new net A2: D10.A, IN2.2, JANALOG.3
- new net A3: D9.A, IN3.2, JANALOG.4
- new net A4: JANALOG.5
- new net A5: JANALOG.6
- new net AREF: JHIGH.8
- new net BRAKEA: BRAKE-A_DISABLE.1, BRAKE-A_DISABLE.2, IC2A.I1, JHIGH.2, RN2B.2
- new net BRAKEB: BRAKE-B_DISABLE.1, BRAKE-B_DISABLE.2, IC2D.I1, JHIGH.1, RN2A.2
- new net DIRA: IC1.IN1, IC2A.I0, JHIGH.5
- new net DIRA#: IC1.IN2, IC2A.O
- new net DIRB: IC1.IN3, IC2D.I0, JHIGH.6
- new net DIRB#: IC1.IN4, IC2D.O
- new net IOREF: D10.K, D9.K, POWER.2
- new net N$1: LED4.C, RN1D.1
- new net N$10: R5.1, U4.2
- new net N$5: IC4A.-IN, RN2D.1, RN3A.1
- new net N$7: IC4B.-IN, RN2C.1, RN3B.1
- new net N$8: R3.1, U1.2
- new net N$9: R4.1, U3.2
- new net OUT1: D1.A, D5.K, IC1.OUT1, LED1.A, LSP4.MP
- new net OUT2: D2.A, D6.K, IC1.OUT2, LED2.A, LSP3.MP
- new net OUT3: D4.A, D8.K, IC1.OUT4, LED4.A, LSP1.MP
- new net OUT4: D3.A, D7.K, IC1.OUT3, LED3.A, LSP2.MP
- new net PWMA: IC1.ENA, JLOW.4
- new net PWMB: IC1.ENB, JHIGH.4
- new net RESET: POWER.3, RESET.1, RESET.2
- new net SCL: JHIGH.10, TWI-IN.4, TWI-OUT.4
- new net SDA: JHIGH.9, TWI-IN.3, TWI-OUT.3
- new net SNS0: IC4A.OUT, JANALOG.1, RN2D.2, SNS0-ENABLE.1, SNS0-ENABLE.2
- new net SNS1: IC4B.OUT, JANALOG.2, RN2C.2, SNS1_ENABLE.1, SNS1_ENABLE.2
- new net SNSA: IC1.SENA, IC4A.+IN, R1.1
- new net SNSB: IC1.SENB, IC4B.+IN, R2.1
- new net VIN: POWER.8, VIN-CONNECT.1
- new net VMOT: C10.1, C11.1, C9.1, D1.K, D2.K, D3.K, D4.K, IC1.VS, LSP5.MP, VIN-CONNECT.2
- net GND: now also C1.2, C10.2, C11.2, C12.2, C2.2, C3.2, C4.2, C5.2, C6.2, C7.2, C8.2, C9.2, D5.A, D6.A, D7.A, D8.A, IC1.GND1, IC1.GND2, IC1.GND3, IC1.GND4, IC1.PAD1, IC1.PAD2, IC1.PAD3, IC2C.I0, IC2C.I1, IC2P.VSS, IC4P.V-, IN2.1, IN3.1, JHIGH.7, JP2.2, JP3.2, LSP6.MP, OUT5.1, OUT6.1, POWER.6, POWER.7, R3.2, R4.2, R5.2, RESET.3, RESET.4, RN1A.2, RN1B.2, RN1C.2, RN1D.2, RN2A.1, RN2B.1, RN3A.2, RN3B.2, TWI-IN.1, TWI-OUT.1, U3.5, U4.5
- net N$2: now also LED3.C, RN1C.1; no longer R1.1, U1.2
- net N$3: now also LED2.C, RN1B.1; no longer JP2.2
- net N$4: now also LED1.C, RN1A.1; no longer R2.1
- net SIG: now also JP2.1, JP3.1, U3.4, U4.4
- net VCC: now also JP2.3, JP3.3, U3.1, U3.3, U4.1, U4.3
Other:
- note added: "12V DC"
- note added: "DEFAULT:Closed"
- note added: "SCL"
- note added: "SDA"
- note added: "VIN Max"
